Commit message: changed_again

File: description/robot_core.xacro (robot description, xacro)
@@ -31,33 +31,34 @@
         </visual>
     </link>
-    <!--LEFT WHEEL LINK-->
-    <joint name="left_wheel_joint" type = "continuous">
-        <parent link= "base_link"/>
+    <!-- LEFT WHEEL -->
+    <joint name="left_wheel_joint" type="continuous">
+        <parent link="base_link"/>
         <child link="left_wheel"/>
-        <origin xyz="0.0 0.175 0" rpy="-${pi/2} 0 0"/>
-        <axis xys = "0 0 1"/>
+        <origin xyz="0 0.175 0" rpy="-${pi/2} 0 0"/>
+        <axis xyz="0 0 1"/>
     </joint>
     <link name="left_wheel">
         <visual>
             <geometry>
-                <cylinder radius="0.05" length="0.04"/>
+                <cylinder length="0.04" radius="0.05" />/>
             </geometry>
             <material name="blue"/>
         </visual>
     </link>
-    <!--right WHEEL LINK-->
-    <joint name="right_wheel_joint" type = "continuous">
-        <parent link= "base_link"/>
-        <child link="right_wheel"/>
-        <origin xyz="0.0 0.175 0" rpy="${pi/2} 0 0"/>
-        <axis xys = "0 0 -1"/>
-    </joint>
-    <link name="right_wheel">
-        <visual>
-            <geometry>
-                <cylinder radius="0.05" length="0.04"/>
-            </geometry>
-            <material name="blue"/>
-        </visual>
-    </link>
+<!-- RIGHT WHEEL -->
+<joint name="right_wheel_joint" type="continuous">
+    <parent link="base_link"/>
+    <child link="right_wheel"/>
+    <origin xyz="0 -0.175 0" rpy="${pi/2} 0 0"/>
+    <axis xyz="0 0 -1"/>
+</joint>
+<link name="right_wheel">
+    <visual>
+        <geometry>
+            <cylinder length="0.04" radius="0.05" />/>
+        </geometry>
+        <material name="blue"/>
+    </visual>
+</link>
+<!-- Castor Wheel Link-->
 </robot>

Commit message: change_name_again

File: description/robot_core.xacro (robot description, xacro)
@@ -1,4 +1,5 @@
 <?xml version="1.0"?>
 <robot xmlns:xacro="http://www.ros.org/wiki/xacro">
+    <xacro:include filename="inertial_macros.xacro"/>
     <material name="white">
         <color rgba="1 1 1 1"/>
@@ -30,6 +31,15 @@
             <material name="white"/>
         </visual>
+        <collision>
+            <origin xyz="0.15 0 0.075" rpy="0 0 0"/>
+            <geometry>
+                <box size="0.3 0.3 0.15"/>
+            </geometry>
+        </collision>
+        <xacro:inertial_box mass= "0.5" x= "0.3" y="0.3" z="0.15">
+            <origin xyz="0.15 0 0.075" rpy="0 0 0"/>
+        </xacro:inertial_box>
     </link>
-    <!-- LEFT WHEEL -->
+    <!-- LEFT WHEEL LINK-->
     <joint name="left_wheel_joint" type="continuous">
         <parent link="base_link"/>
@@ -41,24 +51,61 @@
         <visual>
             <geometry>
-                <cylinder length="0.04" radius="0.05" />/>
+                <cylinder length="0.04" radius="0.05" />
             </geometry>
             <material name="blue"/>
         </visual>
+        <collision>
+            <geometry>
+                <cylinder length="0.04" radius="0.05" />
+            </geometry>
+        </collision>
+        <xacro:inertial_cylinder mass="0.1" length="0.04" radius="0.05">
+            <origin xyz= "0 0 0" rpy = "0 0 0"/>
+        </xacro:inertial_cylinder>
     </link>
-<!-- RIGHT WHEEL -->
-<joint name="right_wheel_joint" type="continuous">
-    <parent link="base_link"/>
-    <child link="right_wheel"/>
-    <origin xyz="0 -0.175 0" rpy="${pi/2} 0 0"/>
-    <axis xyz="0 0 -1"/>
+    <!-- RIGHT WHEEL LINK-->
+    <joint name="right_wheel_joint" type="continuous">
+        <parent link="base_link"/>
+        <child link="right_wheel"/>
+        <origin xyz="0 -0.175 0" rpy="${pi/2} 0 0"/>
+        <axis xyz="0 0 -1"/>
+    </joint>
+    <link name="right_wheel">
+        <visual>
+            <geometry>
+                <cylinder length="0.04" radius="0.05" />
+            </geometry>
+            <material name="blue"/>
+        </visual>
+        <collision>
+            <geometry>
+                <cylinder length="0.04" radius="0.05" />
+            </geometry>
+        </collision>
+        <xacro:inertial_cylinder mass="0.1" length="0.04" radius="0.05">
+            <origin xyz= "0 0 0" rpy = "0 0 0"/>
+        </xacro:inertial_cylinder>
+    </link>
+<!-- CASTER WHEEL LINK-->
+<joint name="caster_wheel_joint" type="fixed">
+    <parent link="chassis"/>
+    <child link="caster_wheel"/>
+    <origin xyz="0.24 0 0" rpy="0 0 0"/>
 </joint>
-<link name="right_wheel">
+<link name="caster_wheel">
     <visual>
         <geometry>
-            <cylinder length="0.04" radius="0.05" />/>
+            <sphere radius="0.05" />
         </geometry>
-        <material name="blue"/>
+        <material name="black"/>
     </visual>
+    <collision>
+        <geometry>
+            <sphere radius="0.05" />
+        </geometry>
+    </collision>
+    <xacro:inertial_sphere mass="0.1" radius = "0.05">
+        <origin xyz= "0 0 0" rpy = "0 0 0"/>
+    </xacro:inertial_sphere>
 </link>
-<!-- Castor Wheel Link-->
 </robot>

Commit message: rviz_and_gazebo_sim_done_without_obstacles_yet

File: description/robot_core.xacro (robot description, xacro)
@@ -41,4 +41,7 @@
         </xacro:inertial_box>
     </link>
+    <gazebo reference="chassis">
+        <material>Gazebo/White</material>
+    </gazebo>
     <!-- LEFT WHEEL LINK-->
     <joint name="left_wheel_joint" type="continuous">
@@ -64,4 +67,7 @@
         </xacro:inertial_cylinder>
     </link>
+    <gazebo reference="left_wheel">
+        <material>Gazebo/Blue</material>
+    </gazebo>
     <!-- RIGHT WHEEL LINK-->
     <joint name="right_wheel_joint" type="continuous">
@@ -87,4 +93,7 @@
         </xacro:inertial_cylinder>
     </link>
+    <gazebo reference="right_wheel">
+        <material>Gazebo/Blue</material>
+    </gazebo>
 <!-- CASTER WHEEL LINK-->
 <joint name="caster_wheel_joint" type="fixed">
@@ -109,3 +118,8 @@
     </xacro:inertial_sphere>
 </link>
+<gazebo reference="caster_wheel">
+    <material>Gazebo/Black</material>
+    <mu1 value="0.001"/>
+    <mu2 value="0.001"/>
+</gazebo>
 </robot>
